File: PCB/EEPROM_MikroBus/EEPROM_MikroBus.kicad_sch (KiCad schematic)
At the start: 5 parts, among them J1 Conn_01x08, J2 Conn_01x08, U1 24FC04_8DIP

Commit message: Added EEPROM PCB Files (Complete)
Parts:
- D1: footprint (none) -> LED_SMD:LED_0603_1608Metric_Pad1.05x0.95mm_HandSolder
- R1: footprint (none) -> Resistor_SMD:R_0603_1608Metric_Pad0.98x0.95mm_HandSolder
Changed lines of the file:
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@@
     (property "Reference" "D1" (id 0) (at 189.5475 115.57 0))
     (property "Value" "LED" (id 1) (at 189.5475 118.11 0))
-    (property "Footprint" "" (id 2) (at 187.96 123.19 0)
+    (property "Footprint" "LED_SMD:LED_0603_1608Metric_Pad1.05x0.95mm_HandSolder" (id 2) (at 187.96 123.19 0)
       (effects (font (size 1.27 1.27)) hide)
     )
@@
     (property "Reference" "R1" (id 0) (at 175.26 116.84 90))
     (property "Value" "R" (id 1) (at 175.26 119.38 90))
-    (property "Footprint" "" (id 2) (at 175.26 124.968 90)
+    (property "Footprint" "Resistor_SMD:R_0603_1608Metric_Pad0.98x0.95mm_HandSolder" (id 2) (at 175.26 124.968 90)
       (effects (font (size 1.27 1.27)) hide)
     )
@@
     )
     (path "/8b704647-5a97-4744-90a6-63daaa7285da"
-      (reference "D1") (unit 1) (value "LED") (footprint "")
+      (reference "D1") (unit 1) (value "LED") (footprint "LED_SMD:LED_0603_1608Metric_Pad1.05x0.95mm_HandSolder")
     )
     (path "/870f9307-d351-46af-8b91-510f1f6d3cd0"
@@
     )
     (path "/fb4d78fe-4c54-4934-9531-b549dbe7b218"
-      (reference "R1") (unit 1) (value "R") (footprint "")
+      (reference "R1") (unit 1) (value "R") (footprint "Resistor_SMD:R_0603_1608Metric_Pad0.98x0.95mm_HandSolder")
     )
     (path "/775a870d-2cec-45d0-80a9-64d920e3da25"
